File: hardware/SF4-hardware/SF4-hardware.kicad_sch (KiCad schematic)
At the start: 7 parts, among them U1 CD4053B, U4 LM324, U5 LM324

Commit message: Final changes to hardware in kicad
Parts:
- R18: value R -> 4.7k
- R19: value R -> 1k
Changed lines of the file:
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@@
 			)
 		)
-		(property "Value" "R"
+		(property "Value" "1k"
 			(at 52.07 153.6699 0)
 			(effects
@@
 			)
 		)
-		(property "Value" "R"
+		(property "Value" "4.7k"
 			(at 52.07 143.5099 0)
 			(effects
